File: keyboardTest.kicad_sch (KiCad schematic)
At the start: 118 parts, among them J1 DRAGON_CONNECTION, SW1 O, SW10 A, SW11 I, SW12 Q, SW13 Y, SW14 Clear, SW15 2, SW16 :, SW17 B, SW18 J, SW19 R, SW2 8, SW20 Z, SW21 Break, SW22 3, SW23 ;, SW24 C, SW25 K, SW26 S, SW27 Up, SW28 4, SW29 ,, SW3 At, SW30 D, SW31 L, SW32 T, SW33 Down, SW34 5, SW35 -, SW36 E, SW37 M, SW38 U, SW39 Left, SW4 H, SW40 6, SW41 ., SW42 F, SW43 N, SW44 V, SW45 Right, SW46 7, SW47 /, SW48 G, SW49 O, SW5 P, SW50 W, SW51 Space, SW52 Shift, SW53 Shift, SW6 X, SW7 Enter, SW8 1, SW9 9

Commit message: rectify spacebar row
Parts:
- added D54, D55: D, Diode_SMD:D_0805_2012Metric, symbol Device:D
- added SW54: Ctrl, Button_Switch_Keyboard:SW_Cherry_MX_1.00u_PCB, symbol Switch:SW_Push
- added SW55: Fn, Button_Switch_Keyboard:SW_Cherry_MX_1.00u_PCB, symbol Switch:SW_Push
- added SWS1: Switch Stabiliser, Mounting_Keyboard_Stabilizer:Stabilizer_Cherry_MX_6.00u, symbol Mechanical:MountingHole
- SW51: footprint Button_Switch_Keyboard:SW_Cherry_MX_6.25u_PCB -> Switch_Keyboard_Cherry_MX:SW_Cherry_MX_PCB_6.00u
Connections:
- net PA5: now also SW51.2; no longer SW51.1
- net PA6: now also SW54.1, SW55.1
- net PB3: now also D54.2 (A)
- net PB6: now also D55.2 (A)
- net at D51.1 (K): now also SW51.1; no longer SW51.2
- new net: D55.1 (K), SW55.2
- new net: D54.1 (K), SW54.2
Changed lines of the file:
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@@
   (junction (at 271.78 102.87) (diameter 0) (color 0 0 0 0)
   )
+  (junction (at 191.516 188.468) (diameter 0) (color 0 0 0 0)
+  )
   (junction (at 226.822 102.87) (diameter 0) (color 0 0 0 0)
   )
@@
   (junction (at 269.2322 198.12) (diameter 0) (color 0 0 0 0)
   )
+  (junction (at 184.15 198.12) (diameter 0) (color 0 0 0 0)
+  )
   (junction (at 250.19 102.87) (diameter 0) (color 0 0 0 0)
   )
@@
   (junction (at 183.896 157.226) (diameter 0) (color 0 0 0 0)
   )
+  (junction (at 250.19 198.12) (diameter 0) (color 0 0 0 0)
+  )
   (junction (at 212.852 167.386) (diameter 0) (color 0 0 0 0)
   )
@@
   (junction (at 212.852 147.828) (diameter 0) (color 0 0 0 0)
   )
+  (junction (at 257.81 188.468) (diameter 0) (color 0 0 0 0)
+  )
   (wire (pts (xy 279.4 208.28) (xy 279.4 229.362))
     (stroke (width 0) (type default))
@@
     (stroke (width 0) (type default))
   )
-  (wire (pts (xy 160.02 198.12) (xy 269.2322 198.12))
+  (wire (pts (xy 191.516 188.468) (xy 191.516 208.2531))
+    (stroke (width 0) (type default))
+  )
+  (wire (pts (xy 160.02 198.12) (xy 184.15 198.12))
     (stroke (width 0) (type default))
   )
@@
     (stroke (width 0) (type default))
   )
+  (wire (pts (xy 184.15 198.0931) (xy 184.15 198.12))
+    (stroke (width 0) (type default))
+  )
   (wire (pts (xy 160.02 157.226) (xy 183.896 157.226))
     (stroke (width 0) (type default))
@@
     (stroke (width 0) (type default))
   )
+  (wire (pts (xy 250.19 198.12) (xy 269.2322 198.12))
+    (stroke (width 0) (type default))
+  )
   (wire (pts (xy 271.78 157.226) (xy 292.608 157.226))
     (stroke (width 0) (type default))
@@
     (stroke (width 0) (type default))
   )
+  (wire (pts (xy 191.516 208.2531) (xy 191.4726 208.2531))
+    (stroke (width 0) (type default))
+  )
   (wire (pts (xy 269.2322 219.202) (xy 269.2322 198.12))
     (stroke (width 0) (type default))
@@
     (stroke (width 0) (type default))
   )
+  (wire (pts (xy 184.15 198.12) (xy 250.19 198.12))
+    (stroke (width 0) (type default))
+  )
   (wire (pts (xy 167.64 70.612) (xy 167.64 96.012))
     (stroke (width 0) (type default))
@@
     (stroke (width 0) (type default))
   )
+  (wire (pts (xy 257.81 188.468) (xy 257.81 208.28))
+    (stroke (width 0) (type default))
+  )
   (wire (pts (xy 90.678 78.74) (xy 88.138 78.74))
     (stroke (width 0) (type default))
@@
   )
   (wire (pts (xy 234.442 113.03) (xy 234.442 130.81))
+    (stroke (width 0) (type default))
+  )
+  (wire (pts (xy 183.8526 198.0931) (xy 184.15 198.0931))
     (stroke (width 0) (type default))
   )
@@
     )
   )
+  (symbol (lib_id "Switch:SW_Push") (at 250.19 203.2 270) (unit 1)
+    (in_bom yes) (on_board yes) (dnp no) (fields_autoplaced)
+    (property "Reference" "SW55" (at 254 202.565 90)
+      (effects (font (size 1.27 1.27)) (justify left))
+    )
+    (property "Value" "Fn" (at 254 205.105 90)
+      (effects (font (size 1.27 1.27)) (justify left))
+    )
+    (property "Footprint" "Button_Switch_Keyboard:SW_Cherry_MX_1.00u_PCB" (at 255.27 203.2 0)
+      (effects (font (size 1.27 1.27)) hide)
+    )
+    (property "Datasheet" "~" (at 255.27 203.2 0)
+      (effects (font (size 1.27 1.27)) hide)
+    )
+    (pin "1")
+    (pin "2")
+    (instances
+      (project "keyboardTest"
+        (path "/f35e9616-f481-4cdb-9e32-caf70bd322dd"
+          (reference "SW55") (unit 1)
+        )
+      )
+    )
+  )
   (symbol (lib_id "Switch:SW_Push") (at 138.938 107.95 270) (unit 1)
     (in_bom yes) (on_board yes) (dnp no) (fields_autoplaced)
@@
     )
   )
+  (symbol (lib_id "Device:D") (at 187.6626 208.2531 0) (mirror x) (unit 1)
+    (in_bom yes) (on_board yes) (dnp no)
+    (property "Reference" "D54" (at 187.6626 211.0471 0)
+      (effects (font (size 1.27 1.27)))
+    )
+    (property "Value" "D" (at 190.7106 211.0471 0)
+      (effects (font (size 1.27 1.27)))
+    )
+    (property "Footprint" "Diode_SMD:D_0805_2012Metric" (at 187.6626 208.2531 0)
+      (effects (font (size 1.27 1.27)) hide)
+    )
+    (property "Datasheet" "~" (at 187.6626 208.2531 0)
+      (effects (font (size 1.27 1.27)) hide)
+    )
+    (property "Sim.Device" "D" (at 187.6626 208.2531 0)
+      (effects (font (size 1.27 1.27)) hide)
+    )
+    (property "Sim.Pins" "1=K 2=A" (at 187.6626 208.2531 0)
+      (effects (font (size 1.27 1.27)) hide)
+    )
+    (pin "1")
+    (pin "2")
+    (instances
+      (project "keyboardTest"
+        (path "/f35e9616-f481-4cdb-9e32-caf70bd322dd"
+          (reference "D54") (unit 1)
+        )
+      )
+    )
+  )
   (symbol (lib_id "Switch:SW_Push") (at 160.02 162.306 270) (unit 1)
     (in_bom yes) (on_board yes) (dnp no) (fields_autoplaced)
@@
         (path "/f35e9616-f481-4cdb-9e32-caf70bd322dd"
           (reference "D18") (unit 1)
+        )
+      )
+    )
+  )
+  (symbol (lib_id "Device:D") (at 254 208.28 0) (mirror x) (unit 1)
+    (in_bom yes) (on_board yes) (dnp no)
+    (property "Reference" "D55" (at 254 211.074 0)
+      (effects (font (size 1.27 1.27)))
+    )
+    (property "Value" "D" (at 257.048 211.074 0)
+      (effects (font (size 1.27 1.27)))
+    )
+    (property "Footprint" "Diode_SMD:D_0805_2012Metric" (at 254 208.28 0)
+      (effects (font (size 1.27 1.27)) hide)
+    )
+    (property "Datasheet" "~" (at 254 208.28 0)
+      (effects (font (size 1.27 1.27)) hide)
+    )
+    (property "Sim.Device" "D" (at 254 208.28 0)
+      (effects (font (size 1.27 1.27)) hide)
+    )
+    (property "Sim.Pins" "1=K 2=A" (at 254 208.28 0)
+      (effects (font (size 1.27 1.27)) hide)
+    )
+    (pin "1")
+    (pin "2")
+    (instances
+      (project "keyboardTest"
+        (path "/f35e9616-f481-4cdb-9e32-caf70bd322dd"
+          (reference "D55") (unit 1)
         )
       )
@@
     )
   )
+  (symbol (lib_id "Switch:SW_Push") (at 183.8526 203.1731 270) (unit 1)
+    (in_bom yes) (on_board yes) (dnp no) (fields_autoplaced)
+    (property "Reference" "SW54" (at 187.6626 202.5381 90)
+      (effects (font (size 1.27 1.27)) (justify left))
+    )
+    (property "Value" "Ctrl" (at 187.6626 205.0781 90)
+      (effects (font (size 1.27 1.27)) (justify left))
+    )
+    (property "Footprint" "Button_Switch_Keyboard:SW_Cherry_MX_1.00u_PCB" (at 188.9326 203.1731 0)
+      (effects (font (size 1.27 1.27)) hide)
+    )
+    (property "Datasheet" "~" (at 188.9326 203.1731 0)
+      (effects (font (size 1.27 1.27)) hide)
+    )
+    (pin "1")
+    (pin "2")
+    (instances
+      (project "keyboardTest"
+        (path "/f35e9616-f481-4cdb-9e32-caf70bd322dd"
+          (reference "SW54") (unit 1)
+        )
+      )
+    )
+  )
   (symbol (lib_id "Switch:SW_Push") (at 271.78 203.2 270) (unit 1)
     (in_bom yes) (on_board yes) (dnp no) (fields_autoplaced)
@@
     )
   )
+  (symbol (lib_id "Mechanical:MountingHole") (at 60.96 209.55 0) (unit 1)
+    (in_bom yes) (on_board yes) (dnp no) (fields_autoplaced)
+    (property "Reference" "SWS1" (at 63.5 208.28 0)
+      (effects (font (size 1.27 1.27)) (justify left))
+    )
+    (property "Value" "Switch Stabiliser" (at 63.5 210.82 0)
+      (effects (font (size 1.27 1.27)) (justify left))
+    )
+    (property "Footprint" "Mounting_Keyboard_Stabilizer:Stabilizer_Cherry_MX_6.00u" (at 60.96 209.55 0)
+      (effects (font (size 1.27 1.27)) hide)
+    )
+    (property "Datasheet" "~" (at 60.96 209.55 0)
+      (effects (font (size 1.27 1.27)) hide)
+    )
+    (instances
+      (project "keyboardTest"
+        (path "/f35e9616-f481-4cdb-9e32-caf70bd322dd"
+          (reference "SWS1") (unit 1)
+        )
+      )
+    )
+  )
   (symbol (lib_id "Device:D") (at 123.444 208.28 0) (mirror x) (unit 1)
     (in_bom yes) (on_board yes) (dnp no)
@@
     )
   )
-  (symbol (lib_id "Switch:SW_Push") (at 271.78 183.388 270) (unit 1)
-    (in_bom yes) (on_board yes) (dnp no) (fields_autoplaced)
-    (property "Reference" "SW51" (at 275.59 182.753 90)
-      (effects (font (size 1.27 1.27)) (justify left))
-    )
-    (property "Value" "Space" (at 275.59 185.293 90)
-      (effects (font (size 1.27 1.27)) (justify left))
-    )
-    (property "Footprint" "Button_Switch_Keyboard:SW_Cherry_MX_6.25u_PCB" (at 276.86 183.388 0)
-      (effects (font (size 1.27 1.27)) hide)
-    )
+  (symbol (lib_id "Switch:SW_Push") (at 271.78 183.388 270) (mirror x) (unit 1)
+    (in_bom yes) (on_board yes) (dnp no)
+    (property "Reference" "SW51" (at 275.59 184.023 90)
+      (effects (font (size 1.27 1.27)) (justify left))
+    )
+    (property "Value" "Space" (at 275.59 181.483 90)
+      (effects (font (size 1.27 1.27)) (justify left))
+    )
+    (property "Footprint" "Switch_Keyboard_Cherry_MX:SW_Cherry_MX_PCB_6.00u" (at 276.86 183.388 0)
+      (effects (font (size 1.27 1.27)) hide)
+    )

Commit message: update pcb for spare stabiliser position
Parts:
- added SWS2: 8u Switch Stabiliser, Mounting_Keyboard_Stabilizer:Stabilizer_Cherry_MX_8.00u, symbol Mechanical:MountingHole
- SWS1: value Switch Stabiliser -> 6u Switch Stabiliser
Changed lines of the file:
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@@
       (effects (font (size 1.27 1.27)) (justify left))
     )
-    (property "Value" "Switch Stabiliser" (at 63.5 210.82 0)
+    (property "Value" "6u Switch Stabiliser" (at 63.5 210.82 0)
       (effects (font (size 1.27 1.27)) (justify left))
     )
@@
         )
       )
+    )
+  )
+  (symbol (lib_id "Mechanical:MountingHole") (at 60.96 217.17 0) (unit 1)
+    (in_bom yes) (on_board yes) (dnp no) (fields_autoplaced)
+    (property "Reference" "SWS2" (at 63.5 215.9 0)
+      (effects (font (size 1.27 1.27)) (justify left))
+    )
+    (property "Value" "8u Switch Stabiliser" (at 63.5 218.44 0)
+      (effects (font (size 1.27 1.27)) (justify left))
+    )
+    (property "Footprint" "Mounting_Keyboard_Stabilizer:Stabilizer_Cherry_MX_8.00u" (at 60.96 217.17 0)
+      (effects (font (size 1.27 1.27)) hide)
+    )
+    (property "Datasheet" "~" (at 60.96 217.17 0)
+      (effects (font (size 1.27 1.27)) hide)
+    )
+    (instances
+      (project "keyboardTest"
+        (path "/f35e9616-f481-4cdb-9e32-caf70bd322dd"
+          (reference "SWS2") (unit 1)
+        )
+      )

Commit message: shrinkify board
Parts:
- removed H1, H2: MountingHole, MountingHole:MountingHole_5.3mm_M5, symbol Mechanical:MountingHole
- H10, H11, H3, H4, H5, H6, H7, H8, H9: now not fitted; now left out of the parts list
Changed lines of the file:
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@@
   )
   (symbol (lib_id "Mechanical:MountingHole") (at 31.75 162.306 0) (unit 1)
-    (in_bom yes) (on_board yes) (dnp no) (fields_autoplaced)
+    (in_bom no) (on_board yes) (dnp yes) (fields_autoplaced)
     (property "Reference" "H3" (at 34.29 161.671 0)
       (effects (font (size 1.27 1.27)) (justify left))
@@
   )
   (symbol (lib_id "Mechanical:MountingHole") (at 61.214 162.052 0) (unit 1)
-    (in_bom yes) (on_board yes) (dnp no) (fields_autoplaced)
+    (in_bom no) (on_board yes) (dnp yes) (fields_autoplaced)
     (property "Reference" "H4" (at 63.754 161.417 0)
       (effects (font (size 1.27 1.27)) (justify left))
@@
   )
   (symbol (lib_id "Mechanical:MountingHole") (at 32.766 176.022 0) (unit 1)
-    (in_bom yes) (on_board yes) (dnp no) (fields_autoplaced)
+    (in_bom no) (on_board yes) (dnp yes) (fields_autoplaced)
     (property "Reference" "H6" (at 35.306 175.387 0)
       (effects (font (size 1.27 1.27)) (justify left))
@@
   )
   (symbol (lib_id "Mechanical:MountingHole") (at 90.17 190.754 0) (unit 1)
-    (in_bom yes) (on_board yes) (dnp no) (fields_autoplaced)
+    (in_bom no) (on_board yes) (dnp yes) (fields_autoplaced)
     (property "Reference" "H11" (at 92.71 190.119 0)
       (effects (font (size 1.27 1.27)) (justify left))
@@
   )
   (symbol (lib_id "Mechanical:MountingHole") (at 33.02 191.516 0) (unit 1)
-    (in_bom yes) (on_board yes) (dnp no) (fields_autoplaced)
+    (in_bom no) (on_board yes) (dnp yes) (fields_autoplaced)
     (property "Reference" "H9" (at 35.56 190.881 0)
       (effects (font (size 1.27 1.27)) (justify left))
@@
     )
   )
-  (symbol (lib_id "Mechanical:MountingHole") (at 59.69 132.588 0) (unit 1)
-    (in_bom yes) (on_board yes) (dnp no) (fields_autoplaced)
-    (property "Reference" "H1" (at 62.23 131.953 0)
-      (effects (font (size 1.27 1.27)) (justify left))
-    )
-    (property "Value" "MountingHole" (at 62.23 134.493 0)
-      (effects (font (size 1.27 1.27)) (justify left))
-    )
-    (property "Footprint" "MountingHole:MountingHole_5.3mm_M5" (at 59.69 132.588 0)
-      (effects (font (size 1.27 1.27)) hide)
-    )
-    (property "Datasheet" "~" (at 59.69 132.588 0)
-      (effects (font (size 1.27 1.27)) hide)
-    )
-    (instances
-      (project "keyboardTest"
-        (path "/f35e9616-f481-4cdb-9e32-caf70bd322dd"
-          (reference "H1") (unit 1)
-        )
-      )
-    )
-  )
   (symbol (lib_id "Switch:SW_Push") (at 160.02 90.932 270) (unit 1)
     (in_bom yes) (on_board yes) (dnp no) (fields_autoplaced)
@@
   )
   (symbol (lib_id "Mechanical:MountingHole") (at 89.662 176.784 0) (unit 1)
-    (in_bom yes) (on_board yes) (dnp no) (fields_autoplaced)
+    (in_bom no) (on_board yes) (dnp yes) (fields_autoplaced)
     (property "Reference" "H8" (at 92.202 176.149 0)
       (effects (font (size 1.27 1.27)) (justify left))
@@
   )
   (symbol (lib_id "Mechanical:MountingHole") (at 89.3819 162.7662 0) (unit 1)
-    (in_bom yes) (on_board yes) (dnp no) (fields_autoplaced)
+    (in_bom no) (on_board yes) (dnp yes) (fields_autoplaced)
     (property "Reference" "H5" (at 91.9219 162.1312 0)
       (effects (font (size 1.27 1.27)) (justify left))
@@
   )
   (symbol (lib_id "Mechanical:MountingHole") (at 60.96 177.038 0) (unit 1)
-    (in_bom yes) (on_board yes) (dnp no) (fields_autoplaced)
+    (in_bom no) (on_board yes) (dnp yes) (fields_autoplaced)
     (property "Reference" "H7" (at 63.5 176.403 0)
       (effects (font (size 1.27 1.27)) (justify left))
@@
     )
   )
-  (symbol (lib_id "Mechanical:MountingHole") (at 59.69 146.304 0) (unit 1)
-    (in_bom yes) (on_board yes) (dnp no) (fields_autoplaced)
-    (property "Reference" "H2" (at 62.23 145.669 0)
-      (effects (font (size 1.27 1.27)) (justify left))
-    )
-    (property "Value" "MountingHole" (at 62.23 148.209 0)
-      (effects (font (size 1.27 1.27)) (justify left))
-    )
-    (property "Footprint" "MountingHole:MountingHole_5.3mm_M5" (at 59.69 146.304 0)
-      (effects (font (size 1.27 1.27)) hide)
-    )
-    (property "Datasheet" "~" (at 59.69 146.304 0)
-      (effects (font (size 1.27 1.27)) hide)
-    )
-    (instances
-      (project "keyboardTest"
-        (path "/f35e9616-f481-4cdb-9e32-caf70bd322dd"
-          (reference "H2") (unit 1)
-        )
-      )
-    )
-  )
   (symbol (lib_id "Switch:SW_Push") (at 226.822 162.306 270) (unit 1)
     (in_bom yes) (on_board yes) (dnp no) (fields_autoplaced)
@@
   )
   (symbol (lib_id "Mechanical:MountingHole") (at 61.468 192.024 0) (unit 1)
-    (in_bom yes) (on_board yes) (dnp no) (fields_autoplaced)
+    (in_bom no) (on_board yes) (dnp yes) (fields_autoplaced)
     (property "Reference" "H10" (at 64.008 191.389 0)
       (effects (font (size 1.27 1.27)) (justify left))
